Commit message: Demo version

File: ros2_ws/src/mtp_gridmap/urdf/robot.urdf (robot description, URDF)
Before this commit: robot mtp_robot, 3 links, 2 joints
Links:
- added link camera_link; visual cylinder length=0.02 radius=0.05
Joints:
- removed joint base_to_gps_joint
- added joint base_to_camera_joint: type fixed, parent base_link, child camera_link, origin xyz=0.16 0.0 0.9 rpy=0 0 0
- added joint base_to_gnss_joint: type fixed, parent base_link, child gnss_link, origin xyz=-0.13 0.0 0.9 rpy=0 0 0
- joint base_to_imu_joint: origin xyz=0 0.1 0  rpy=0 0 0 -> xyz=0 0.0 0.9 rpy=0 0 0
